Commit message: Ajusta orientación del robot y guarda vista con ejes en RViz

File: src/robot_description/urdf/robot.urdf (robot description, URDF)
Before this commit: robot leakscout, 3 links, 2 joints
Links:
- added link cad_link; visual mesh filename=package://robot_description/meshes/chasis.STL scale=0.001 0.001 0.001
- link base_link: geometry 
Joints:
- added joint base_to_cad: type fixed, parent base_link, child cad_link, origin xyz=0 0 0 rpy=0 0 -1.57079632679
- joint wheel_left_joint: parent base_link -> cad_link
- joint wheel_right_joint: parent base_link -> cad_link

Commit message: Integra Colmibot en Gazebo con control PS4

File: src/robot_description/urdf/robot.urdf (robot description, URDF)
Before this commit: robot leakscout, 4 links, 3 joints
Links:
- removed link cad_link
- removed link wheel_left
- removed link wheel_right
- added link wheel_left_link, mass 0.0193581; collision cylinder length=0.006 radius=0.030; visual mesh filename=package://robot_description/meshes/rueda_izquierda.STL scale=0.001 0.001 0.001
- added link wheel_right_link, mass 0.0193581; collision cylinder length=0.006 radius=0.030; visual mesh filename=package://robot_description/meshes/rueda_derecha.STL scale=0.001 0.001 0.001
- link base_link: mass None -> 2.2407514; geometry collision box size=0.180 0.160 0.120; collision sphere radius=0.0079375
Joints:
- removed joint base_to_cad
- joint wheel_left_joint: axis 1 0 0 -> 0 1 0; child wheel_left -> wheel_left_link; limit (none) -> effort=5.0 velocity=30.0; origin xyz=-0.08904754 0 0.0165 rpy=0 0 0 -> xyz=0 0.0890475 0.0165 rpy=0 0 0; parent cad_link -> base_link
- joint wheel_right_joint: axis 1 0 0 -> 0 1 0; child wheel_right -> wheel_right_link; limit (none) -> effort=5.0 velocity=30.0; origin xyz=0.08904754 0 0.0165 rpy=0 0 0 -> xyz=0 -0.0890475 0.0165 rpy=0 0 0; parent cad_link -> base_link
